File: Eagle/CPU/Schaltplan.brd (EAGLE design)
At the start: 105.1 x 85.7 mm, 36 parts, among them IC1 Adress-Dekoder (GAL16V8), IC2 Controller (AT89S52), IC3 Latch (74HC573), IC4 RAM (6264), IC6 7805, Q1 20MHz, X2 MA2X3 (ISP), X3 LED Matrix 0, X5 LED Matrix 1, X6 LED Matrix 2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

Commit message: Further Board allign
Parts:
- removed D2: (no value), 89S52mini:LED3-2,5
- removed R3: 1k8, 89S52mini:R-10
- removed X5: LED Matrix 1, 89S52mini:MA10X2
- removed X6: LED Matrix 2, 89S52mini:MA10X2
- moved R4 154.5 mm to (70.2, 6.67), turned to 270 degrees
- moved C7 149.4 mm to (75.2, 44.1), turned to 90 degrees
- moved C8 140.4 mm to (64.1, 60.0), turned to 270 degrees
- moved D1 115.4 mm to (64.8, 15.9), turned to 180 degrees
- moved C9 99.1 mm to (9.53, 47.6), turned to 90 degrees
- moved X3 53.6 mm to (47.6, 78.7), turned to 0 degrees
- moved C2 31.1 mm to (75.9, 34.0), turned to 270 degrees
- moved IC1 24.1 mm to (57.8, 45.1)
- moved Q1 16.9 mm to (75.9, 25.4), turned to 270 degrees
- moved C1 12.8 mm to (75.9, 16.2)
- moved X7 6.55 mm to (56.5, 7.30)
- moved X2 3.55 mm to (38.1, 7.30), turned to 180 degrees
- moved X8 1.59 mm to (19.7, 7.30)
- moved X1 1.59 mm to (10.8, 24.4), turned to 0 degrees
- moved R1 0.63 mm to (10.8, 15.2)
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Connections:
- removed net !CS1: IC1.16, X5.17
- removed net !CS2: IC1.15, X6.17
- removed net N$2: D2.A, R3.2
- new net N$20: IC1.1
- new net N$5: IC1.13
- new net N$6: IC1.12
- net !CS0: no longer IC1.17
- net !OE: now also IC1.18; no longer IC1.19
- net !RD: now also IC1.5; no longer IC1.7
- net !WE: now also IC1.14; no longer IC1.18
- net !WR: now also IC1.4; no longer IC1.6
- net +5V: no longer R3.1
- net A0: no longer X5.8, X6.8
- net A1: no longer X5.10, X6.10
- net A10: now also IC1.19, IC1.7
- net A11: now also IC1.17, IC1.6
- net A14: no longer IC1.4
- net A15: no longer IC1.5
- net A2: no longer X5.12, X6.12
- net A3: no longer X5.14, X6.14
- net A4: no longer X5.16, X6.16
- net A5: no longer X5.18, X6.18
- net A6: no longer X5.20, X6.20
- net A7: now also IC1.2; no longer IC1.1
- net A8: now also IC1.15, IC1.9; no longer IC1.2
- net A9: now also IC1.16, IC1.8
- net D0: no longer X5.1, X6.1
- net D1: no longer X5.3, X6.3
- net D2: no longer X5.5, X6.5
- net D3: no longer X5.7, X6.7
- net D4: no longer X5.9, X6.9
- net D5: no longer X5.11, X6.11
- net D6: no longer X5.13, X6.13
- net D7: no longer X5.15, X6.15
- net GND: no longer IC1.11, X5.2, X5.4, X6.2, X6.4
- net PT1: no longer D2.C
Routing:
- net +5V: track 304.0 -> 402.9 mm, vias 2 -> 0
- net GND: track 252.5 -> 340.1 mm, vias 2 -> 6
- net A12: track 67.9 -> 0.00 mm
- net A7: track 109.2 -> 55.9 mm, vias 0 -> 2
- net A15: track 51.4 -> 0.00 mm
- net A14: track 43.8 -> 0.00 mm
- net D0: track 65.9 -> 33.7 mm
- net !OE: track 41.9 -> 9.93 mm
- net A5: track 39.4 -> 70.6 mm, vias 0 -> 2
- net D7: track 21.5 -> 51.8 mm
- net D3: track 21.5 -> 51.7 mm
- net A13: track 36.2 -> 6.77 mm
- net D6: track 21.5 -> 49.2 mm
- net D4: track 21.5 -> 48.5 mm
- net D5: track 21.5 -> 48.5 mm
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
Commit message: All connected, check schematics
Parts:
- added X5: (no value), 89S52mini:J1X2
- moved C10 170.8 mm to (70.8, 22.9), turned to 90 degrees
- moved X2 1.27 mm to (38.1, 8.57)
- moved X7 1.27 mm to (56.5, 8.57)
- moved X8 1.27 mm to (19.7, 8.57)
- moved IC1 0.64 mm to (58.4, 45.1)
- moved R4 0.45 mm to (70.5, 6.35)
- moved X3 0.32 mm to (47.6, 79.1)
- moved X1 0.32 mm to (10.5, 24.4)
Connections:
- removed net N$20: IC1.1
- removed net N$5: IC1.13
- removed net N$6: IC1.12
- new net !CS1: IC1.13, X5.1
- new net !CS2: IC1.12, X5.2
- net !CS0: now also IC1.14
- net !WE: now also IC1.15; no longer IC1.14
- net A8: no longer IC1.15, IC1.9
Routing:
- net A12: track 0.00 -> 124.9 mm, vias 0 -> 4
- net A2: track 32.5 -> 110.4 mm, vias 0 -> 2
- net A4: track 32.5 -> 78.3 mm, vias 0 -> 4
- net +5V: track 402.9 -> 441.5 mm, vias 0 -> 2
- net !CS0: track 0.00 -> 38.6 mm, vias 0 -> 2
- net D0: track 33.7 -> 69.1 mm, vias 0 -> 4
- net GND: track 340.1 -> 361.2 mm, vias 6 -> 10
- net A8: track 26.4 -> 45.0 mm, vias 0 -> 2
- net A6: track 32.5 -> 47.8 mm
- net A1: track 32.6 -> 47.4 mm
- net A3: track 32.5 -> 46.7 mm
- net D2: track 53.8 -> 67.1 mm, vias 0 -> 4
- net D1: track 60.8 -> 70.0 mm, vias 0 -> 2
- net A0: track 45.4 -> 54.6 mm
- net A5: track 70.6 -> 79.5 mm
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