File: Eagle/CPU/Schaltplan.sch (EAGLE design)
At the start: 25 parts, among them IC1 Adress-Dekoder (GAL16V8), IC2 Controller (AT89S52), IC3 Latch (74HC573), IC4 RAM (6264), IC6 7805, Q1 20MHz, X2 MA2X3 (ISP), X3 LED Matrix 0, X5 LED Matrix 1, X6 LED Matrix 2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

Commit message: Connect Input devices and clean up a bit, some ERC fixes aswell
Parts:
- removed D1: (no value), 89S52mini:LED3-2,5
Connections:
- new net ISP0: IC2.P1.5, X2.4
- new net ISP1: IC2.P1.6, X2.1
- new net ISP2: IC2.P1.7, X2.3
- new net PAD2: X8.5
- new net PAD4: X8.1
- new net PT1: X7.13
- new net PT2: X7.11
- new net PT4: X7.7
- net +5V: now also IC2.VCC, IC4.VCC, X7.14, X7.16, X8.14, X8.16
- net A8: now also IC1.I5
- net GND: now also IC2.GND, X7.2, X7.4, X8.2, X8.4
- net PAD0: now also X8.9
- net PAD1: now also X8.7
- net PAD3: now also X8.3
- net PT0: now also X7.15
- net PT3: now also X7.9
- net PT5: now also X7.5
Other:
- moved on the sheet: C3, R1, R2, S1, X1, X2, X7, X8

Commit message: finish schema and start with board
Parts:
- added C10, C7, C8, C9: 100n, 89S52mini:C-2,5
- added D1, D2: (no value), 89S52mini:LED3-2,5
- added P1, P2, P3, P4: (no value), 89S52mini:MPAD-3,0
- added R3, R4: 1k8, 89S52mini:R-10
Connections:
- new net N$1: D1.A, R4.1
- new net N$2: D2.A, R3.2
- net !RD: now also IC1.I6; no longer IC1.I2
- net !WR: now also IC1.I5; no longer IC1.I1
- net +5V: now also C10.2, C7.2, C8.2, C9.2, IC2.\!EA, R3.1, R4.2
- net A13: now also IC1.I2; no longer IC1.I6
- net A14: now also IC1.I3; no longer IC1.I7
- net A15: now also IC1.I4; no longer IC1.I8
- net A7: now also IC1.I0/CLK; no longer IC1.I4
- net A8: now also IC1.I1; no longer IC1.I5
- net GND: now also C10.1, C7.1, C8.1, C9.1, IC4.GND
- net PAD2: now also IC2.P1.2
- net PAD4: now also IC2.P1.4
- net PT1: now also D2.C, IC2.P3.1
- net PT2: now also IC2.P3.2
- net PT4: now also IC2.P3.4
- net PT5: now also D1.C

Commit message: Further Board allign
Parts:
- removed D2: (no value), 89S52mini:LED3-2,5
- removed R3: 1k8, 89S52mini:R-10
- removed X5: LED Matrix 1, 89S52mini:MA10X2
- removed X6: LED Matrix 2, 89S52mini:MA10X2
Connections:
- removed net !CS1: IC1.IOQ3, X5.17
- removed net !CS2: IC1.IOQ4, X6.17
- removed net N$2: D2.A, R3.2
- new net N$20: IC1.I0/CLK
- new net N$5: IC1.IOQ6
- new net N$6: IC1.IOQ7
- net !CS0: no longer IC1.IOQ2
- net !OE: now also IC1.IOQ1; no longer IC1.IOQ0
- net !RD: now also IC1.I4; no longer IC1.I6
- net !WE: now also IC1.IOQ5; no longer IC1.IOQ1
- net !WR: now also IC1.I3; no longer IC1.I5
- net +5V: no longer R3.1
- net A0: no longer X5.8, X6.8
- net A1: no longer X5.10, X6.10
- net A10: now also IC1.I6, IC1.IOQ0
- net A11: now also IC1.I5, IC1.IOQ2
- net A14: no longer IC1.I3
- net A15: no longer IC1.I4
- net A2: no longer X5.12, X6.12
- net A3: no longer X5.14, X6.14
- net A4: no longer X5.16, X6.16
- net A5: no longer X5.18, X6.18
- net A6: no longer X5.20, X6.20
- net A7: now also IC1.I1; no longer IC1.I0/CLK
- net A8: now also IC1.I8, IC1.IOQ4; no longer IC1.I1
- net A9: now also IC1.I7, IC1.IOQ3
- net D0: no longer X5.1, X6.1
- net D1: no longer X5.3, X6.3
- net D2: no longer X5.5, X6.5
- net D3: no longer X5.7, X6.7
- net D4: no longer X5.9, X6.9
- net D5: no longer X5.11, X6.11
- net D6: no longer X5.13, X6.13
- net D7: no longer X5.15, X6.15
- net GND: no longer IC1.I9/\!OE, X5.2, X5.4, X6.2, X6.4
- net PT1: no longer D2.C

Commit message: All connected, check schematics
Parts:
- added X5: (no value), 89S52mini:J1X2
Connections:
- removed net N$20: IC1.I0/CLK
- removed net N$5: IC1.IOQ6
- removed net N$6: IC1.IOQ7
- new net !CS1: IC1.IOQ6, X5.1
- new net !CS2: IC1.IOQ7, X5.2
- net !CS0: now also IC1.IOQ5
- net !WE: now also IC1.IOQ4; no longer IC1.IOQ5
- net A8: no longer IC1.I8, IC1.IOQ4
