File: KiCad/AdapterBoard/AdapterBoard.kicad_sch (KiCad schematic)
At the start: 5 parts, among them X1 MA10X2, X2 J1X2, X3 MA10X2, X4 MA10X2, X5 MA10X2

Commit message: Screen driver working
Parts:
- X1, X3, X4, X5: footprint 89S52mini_MA10X2 -> Connector_PinHeader_2.54mm:PinHeader_2x10_P2.54mm_Vertical
- X2: footprint 89S52mini_J1X2 -> Connector_PinHeader_2.54mm:PinHeader_1x02_P2.54mm_Vertical
